File: pcb/d4r-ii-cradle.kicad_pcb (KiCad board)
At the start: 2 copper layers, 36 x 36 mm, 17 parts, among them P1 CONN_02X06, P2 CONN_01X01

Commit message: v2 of D4R-II cradle that adds telemetry inverter and buzzer
Parts:
- removed the G*** at (140.8, 95.1) (x2)
- added C1: C, Capacitors_SMD:C_1206_HandSoldering, F.Cu at (153.5, 107.8)
- added G***: LOGO, chickadee:chickadee_2mm_fcu, B.Cu at (138.1, 121.2)
- added G***: LOGO, chickadee:chickadee_2mm_fcu, F.Cu at (138.1, 121.2)
- added G***: LOGO, flightstack:flightstack-8mm, F.Cu at (161.7, 119.6)
- added P3: CONN_01X02, Pin_Headers:Pin_Header_Angled_1x02, F.Cu at (140.4, 92.1)
- added Q1: Q_NMOS_GSD, TO_SOT_Packages_SMD:SOT-23_Handsoldering, F.Cu at (156.0, 122.1)
- added Q2: Q_NMOS_GSD, TO_SOT_Packages_SMD:SOT-23_Handsoldering, F.Cu at (137.3, 93.3)
- added R1: 10k, Resistors_SMD:R_0603_HandSoldering, F.Cu at (153.9, 119.0)
- P2: value CONN_01X01 -> CONN_01X04; footprint Pin_Headers:Pin_Header_Angled_1x01 -> Pin_Headers:Pin_Header_Straight_1x04
- PORT_IN1: footprint DF40-80pin-Header -> hirose-df40:DF40-80pin-Header
- PORT_OUT1: footprint DF40-3-4mm-80pin-Receptacle -> hirose-df40:DF40-3-4mm-80pin-Receptacle
- moved P2 7.62 mm to (142.8, 121.0)
Connections:
- net /ExpansionPort/3V3_0.3A_LL renamed +3V3
- net /ExpansionPort/si2c_SCL renamed /ExpansionPort/i2c_SCL
- net /ExpansionPort/si2c_SDA renamed /ExpansionPort/i2c_SDA
- P2 pad 1: /ExpansionPort/UART1_TX -> GNDPWR
- PORT_IN1 pad 10: /ExpansionPort/xi2c1_SCL -> /ExpansionPort/GPIO6
- PORT_IN1 pad 18: /ExpansionPort/+BATT -> /ExpansionPort/BATT_DIV
- PORT_IN1 pad 9: /ExpansionPort/xi2c1_SDA -> /ExpansionPort/GPIO5
- PORT_OUT1 pad 10: /ExpansionPort/xi2c1_SCL -> Net-(PORT_OUT1-Pad10)
- PORT_OUT1 pad 18: /ExpansionPort/+BATT -> /ExpansionPort/BATT_DIV
- PORT_OUT1 pad 5: /ExpansionPort/GPIO1 -> /ExpansionPort/GPIO2
- PORT_OUT1 pad 6: /ExpansionPort/GPIO2 -> /ExpansionPort/GPIO3
- PORT_OUT1 pad 7: /ExpansionPort/GPIO3 -> /ExpansionPort/GPIO4
- PORT_OUT1 pad 8: /ExpansionPort/GPIO4 -> /ExpansionPort/GPIO5
- PORT_OUT1 pad 9: /ExpansionPort/xi2c1_SDA -> /ExpansionPort/GPIO6
Routing:
- net /ExpansionPort/BATT_DIV: track 0.00 -> 37.3 mm, vias 0 -> 1
- net +3V3: track 36.2 -> 60.6 mm, vias 6 -> 8
- net +5V: track 43.4 -> 65.0 mm
- net /ExpansionPort/GPIO1: track 8.44 -> 28.3 mm, vias 1 -> 3
- net GNDPWR: track 73.2 -> 83.6 mm, vias 11 -> 13
- net /ExpansionPort/xi2c1_SDA: track 8.54 -> 0.00 mm, vias 1 -> 0
- net /ExpansionPort/GPIO5: track 0.00 -> 8.46 mm, vias 0 -> 1
- net /ExpansionPort/xi2c1_SCL: track 7.09 -> 0.00 mm, vias 1 -> 0
- net /ExpansionPort/GPIO6: track 0.00 -> 6.83 mm, vias 0 -> 1
- net /nTELEM: track 0.00 -> 6.19 mm
- net /ExpansionPort/+BATT: track 3.51 -> 0.00 mm, vias 1 -> 0
- net Net-(P3-Pad1): track 0.00 -> 3.13 mm
- net /ExpansionPort/UART1_TX: track 12.0 -> 10.0 mm
- net /ExpansionPort/NEW_HEIGHT_2: track 16.6 -> 14.7 mm
- net /ExpansionPort/TIM1: track 14.6 -> 14.1 mm, vias 2 -> 3
Other:
- board text added: "+5V"
- board text added: "4mm"
- board text added: "5V"
- board text added: "A"
- board text added: "Buzzer"
- board text added: "G"
- board text added: "NC"
- board text added: "RX"
- board text added: "ckd.tech/d4r-ii-c/v2"
- board text removed: "Place D4R-II right side up."
- board text removed: "Telemetry"
- board text removed: "ckd.tech/d4r-ii-c/v1"
